Commit message: introduced new robotic cell for manipulation_example package

File: manipulation_ur5_cell_descriptions/urdf/fixed_parts.xacro (robot description, xacro)
@@ -19,5 +19,5 @@
 <link name="floor">
   <collision>
-    <origin  xyz="0.0 0.0 -0.5" rpy="0 0 0" />
+    <origin  xyz="0.0 0.0 -1.0" rpy="0 0 0" />
     <geometry>
       <box size="8 8 1.0"/>
@@ -39,7 +39,4 @@
     <static>true</static>
 </gazebo>
-<gazebo reference="table">
-    <static>true</static>
-</gazebo>
 </xacro:macro>
 </robot>

File: manipulation_ur5_cell_descriptions/urdf/shopdesk_dim.urdf.xacro (robot description, xacro)
@@ -21,7 +21,7 @@
     </inertial>
     <collision>
-      <origin xyz="0 0 -0.8" rpy="0 0 0" />
+      <origin xyz="0 0 -0.5" rpy="0 0 0" />
       <geometry>
-        <box size="2.04 0.84 1.6"/>
+        <box size="2.0 0.8 1.0"/>
       </geometry>
       <material name="sabbia">
