Commit message: new demonstration cell derived from CNR-STIIMA cella1

File: manipulation_ur5_cell_descriptions/urdf/cell_ur5.xacro (robot description, xacro)
@@ -1,10 +1,8 @@
 <?xml version="1.0"?>
 <robot xmlns:xacro="http://ros.org/wiki/xacro" name="static_cell" >
-<xacro:include filename="$(find cella1_descriptions)/urdf/fixed_parts.xacro" />
+<xacro:include filename="$(find manipulation_ur5_cell_descriptions)/urdf/fixed_parts.xacro" />
 <xacro:static_cell/>
-<xacro:include filename="$(find cella1_descriptions)/urdf/ur5.xacro" />
+<xacro:include filename="$(find manipulation_ur5_cell_descriptions)/urdf/ur5.xacro" />
 <xacro:ur5dimo/>
-<xacro:include filename="$(find cella1_descriptions)/urdf/ur10.xacro" />
-<xacro:ur10dimo/>
 <gazebo>
   <plugin name="ros_control" filename="libgazebo_ros_control.so">

File: manipulation_ur5_cell_descriptions/urdf/conveyor_system.urdf.xacro (robot description, xacro)
@@ -23,5 +23,5 @@
         <geometry>
           <mesh
-            filename="package://cella1_descriptions/meshes/conveyor_system.dae" />
+            filename="package://manipulation_ur5_cell_descriptions/meshes/conveyor_system.dae" />
         </geometry>
         <material

File: manipulation_ur5_cell_descriptions/urdf/fixed_parts.xacro (robot description, xacro)
@@ -2,41 +2,13 @@
 <robot xmlns:xacro="http://ros.org/wiki/xacro" name="static_cell" >
 <xacro:macro name="static_cell">
-<xacro:include filename="$(find cella1_descriptions)/urdf/conveyor_system.urdf.xacro" />
+<xacro:include filename="$(find manipulation_ur5_cell_descriptions)/urdf/conveyor_system.urdf.xacro" />
 <xacro:conveyor_system/>
-<xacro:include filename="$(find cella1_descriptions)/urdf/shopdesk_dim.urdf.xacro" />
+<xacro:include filename="$(find manipulation_ur5_cell_descriptions)/urdf/shopdesk_dim.urdf.xacro" />
 <xacro:shopdesk/>
-<xacro:include filename="$(find cella1_descriptions)/urdf/swiss_cameras.urdf.xacro" />
-<xacro:swisscameras/>
-<xacro:include filename="$(find cella1_descriptions)/urdf/wheeled_table_dim.urdf.xacro" />
-<xacro:wheeled_table_dim/>
 <link name="world" />
-<!--<link name="rs1_depth_optical_frame" />
-<joint name="rs1_depth_optical_frame_fixed" type="fixed">
-  <parent link = "ur10_base_link" />
-  <child  link = "rs1_depth_optical_frame" />
-<origin xyz="-2.814 -0.264 0.528" rpy="-1.686 0.043 -1.279" />
-</joint>
-<link name="rs2_depth_optical_frame" />
-<joint name="rs2_depth_optical_frame_fixed" type="fixed">
-  <parent link = "ur10_base_link" />
-  <child  link = "rs2_depth_optical_frame" />
-<origin xyz="-2.908  1.279  0.489" rpy="-1.556 0.002 -1.876" />
-</joint>-->
-<link name="logi_c270_cella1_notcal" />
-<joint name="logi_c270_cella1_notcal_fixed" type="fixed">
-  <parent link = "world" />
-  <child  link = "logi_c270_cella1_notcal" />
-<origin xyz="1.5 1.5 3.074" rpy="3.074 -0.116 1.368" />
-</joint>
-<link name="logi_c270_cella1" />
-<joint name="logi_c270_cella1_fixed" type="fixed">
-  <parent link = "world" />
-  <child  link = "logi_c270_cella1" />
-  <origin xyz="-1.04 0.36 -0.42" rpy="0 0 -0.22" />
-</joint>
 <joint name="conveyor_system_fixed" type="fixed">
   <parent link = "world" />
   <child  link = "conveyor_system" />
-<origin xyz="-0.92 -0.05 0.99" rpy="0.0 0.0 0.02" />
+<origin xyz="-1.25 -0.05 0.78" rpy="0.0 0.0 0.02" />
 </joint>
 <joint name="shopdesk_fixed" type="fixed">
@@ -44,14 +16,4 @@
   <child  link = "shopdesk" />
 <origin xyz="-0.62 1.55 0.94" rpy="0.0 0.0 ${-0.5*pi}" />
-</joint>
-<joint name="sr_fixed" type="fixed">
-  <parent link = "world" />
-  <child  link = "sr_frame" />
-<origin xyz="3.3 0.8 ${3.068}" rpy="${pi} 0.0 ${-0.5*pi} " />
-</joint>
-<joint name="tabletop_fixed" type="fixed">
-  <parent link = "world" />
-  <child  link = "tabletop" />
-  <origin xyz="1.73 1.72 1.04" rpy="0 0 ${-0.5*pi}" />
 </joint>
 <link name="floor">
@@ -68,43 +30,4 @@
 <origin xyz="2 2 1.0" rpy="0 0 0.0" />
 </joint>
-<link name="wall1">
-  <collision>
-    <origin  xyz="0.0 0.5 1.5" rpy="0 0 0" />
-    <geometry>
-      <box size="8 1 1.5"/>
-    </geometry>
-  </collision>
-</link>
-<joint name="wall1_joint" type="fixed">
-  <parent link = "world" />
-  <child  link = "wall1" />
-<origin xyz="2 3.5 0" rpy="0 0 0.0" />
-</joint>
-<link name="wall2">
-  <collision>
-    <origin  xyz="0.0 -0.5 1.5" rpy="0 0 0" />
-    <geometry>
-      <box size="8 1 1.5"/>
-    </geometry>
-  </collision>
-</link>
-<joint name="wall2_joint" type="fixed">
-  <parent link = "world" />
-  <child  link = "wall2" />
-<origin xyz="2 -1 0" rpy="0 0 0.0" />
-</joint>
-<link name="wall3">
-  <collision>
-    <origin  xyz="-0.5 0.0  1.5" rpy="0 0 0" />
-    <geometry>
-      <box size="1 8  1.5"/>
-    </geometry>
-  </collision>
-</link>
-<joint name="wall3_joint" type="fixed">
-  <parent link = "world" />
-  <child  link = "wall3" />
-<origin xyz="-0.3 2 0" rpy="0 0 0.0" />
-</joint>
 <gazebo reference="world">
     <static>true</static>
@@ -116,7 +39,4 @@
     <static>true</static>
 </gazebo>
-<gazebo reference="tabletop">
-    <static>true</static>
-</gazebo>
 <gazebo reference="table">
     <static>true</static>

File: manipulation_ur5_cell_descriptions/urdf/ur5.xacro (robot description, xacro)
@@ -2,21 +2,12 @@
 <robot xmlns:xacro="http://ros.org/wiki/xacro" name="ur5dimo" >
 <xacro:macro name="ur5dimo">
-<xacro:include filename="$(find cella1_descriptions)/urdf/palmo.urdf.xacro" />
-<xacro:palmo/>
-<xacro:include filename="$(find cella1_descriptions)/urdf/elmo_linear_guide.urdf.xacro" />
-<xacro:elmo_linear_guide/>
 <xacro:arg name="transmission_hw_interface" default="hardware_interface/PositionJointInterface"/>
-<xacro:arg name="kinematics_config_ur5" default="$(find cella1_descriptions)/config/ur5_calib.yaml"/>
+<xacro:arg name="kinematics_config_ur5" default="$(find manipulation_ur5_cell_descriptions)/config/ur5_calib.yaml"/>
 <xacro:include filename="$(find robotiq_ft_sensor)/urdf/robotiq_ft300.urdf.xacro" />
 <xacro:include filename="$(find robotiq_2f_85_gripper_visualization)/urdf/robotiq_arg2f_85_model_macro.xacro" />
-<joint name="elmo_linear_guide_fixed" type="fixed">
-  <parent link = "world" />
-  <child  link = "elmo_linear_guide_stator" />
-  <origin xyz="0.090 -0.32 0.95" rpy="0 0 0.005" />
-</joint>
 <joint name="ur5_joint" type="fixed">
-  <parent link="elmo_linear_guide_cursor" />
+  <parent link="shopdesk" />
   <child  link = "ur5_base_link" />
-  <origin xyz="0.02    0.02   0" rpy="0 0 ${0*pi-0.2}" />
+  <origin xyz="0.7    -0.2   0.0" rpy="0 0 ${0*pi-0.2}" />
 </joint>
 <xacro:include filename="$(find ur_description)/urdf/inc/ur5_macro.xacro"/>
@@ -27,11 +18,6 @@
   <origin xyz="0 0 0" rpy="0 0 0"/>
 </xacro:robotiq_ft300>
-<joint name="palmo_joint" type="fixed">
-  <parent link="ft300_sensor" />
-  <child  link = "palmo" />
-  <origin xyz="0.0    0.0   0" rpy="0 ${pi} 0" />
-</joint>
 <joint name="robotiq_joint" type="fixed">
-<parent link="palmo" />
+<parent link="ur5_tool0" />
 <child link = "robotiq_arg2f_base_link" />
 <origin xyz="0.0 0.0 0.0" rpy="0 0 ${0.0*pi}" />
@@ -40,5 +26,5 @@
 <link name="tip" />
 <joint name="tip_joint" type="fixed">
-  <parent link="palmo" />
+  <parent link="ur5_tool0" />
   <child  link = "tip" />
   <origin xyz="0 0 0.2078" rpy="0 0 0" />

Commit message: wip on new examples

File: manipulation_ur5_cell_descriptions/urdf/cell_ur5.xacro (robot description, xacro)
@@ -4,5 +4,5 @@
 <xacro:static_cell/>
 <xacro:include filename="$(find manipulation_ur5_cell_descriptions)/urdf/ur5.xacro" />
-<xacro:ur5dimo/>
+<!--xacro:ur5dimo/-->
 <gazebo>
   <plugin name="ros_control" filename="libgazebo_ros_control.so">

File: manipulation_ur5_cell_descriptions/urdf/fixed_parts.xacro (robot description, xacro)
@@ -10,5 +10,5 @@
   <parent link = "world" />
   <child  link = "conveyor_system" />
-<origin xyz="-1.25 -0.05 0.78" rpy="0.0 0.0 0.02" />
+<origin xyz="-1.25 -0.05 0.78" rpy="0.0 0.0 0.0" />
 </joint>
 <joint name="shopdesk_fixed" type="fixed">
@@ -28,5 +28,5 @@
   <parent link = "world" />
   <child  link = "floor" />
-<origin xyz="2 2 1.0" rpy="0 0 0.0" />
+<origin xyz="2 2 0.0" rpy="0 0 0.0" />
 </joint>
 <gazebo reference="world">

File: manipulation_ur5_cell_descriptions/urdf/ur5.xacro (robot description, xacro)
@@ -1,18 +1,22 @@
 <?xml version="1.0"?>
 <robot xmlns:xacro="http://ros.org/wiki/xacro" name="ur5dimo" >
-<xacro:macro name="ur5dimo">
+<!--xacro:macro name="ur5dimo"-->
 <xacro:arg name="transmission_hw_interface" default="hardware_interface/PositionJointInterface"/>
 <xacro:arg name="kinematics_config_ur5" default="$(find manipulation_ur5_cell_descriptions)/config/ur5_calib.yaml"/>
+<xacro:arg name="joint_limits_config_ur5" default="$(find manipulation_ur5_cell_descriptions)/config/joint_limits.yaml"/>
 <xacro:include filename="$(find robotiq_ft_sensor)/urdf/robotiq_ft300.urdf.xacro" />
 <xacro:include filename="$(find robotiq_2f_85_gripper_visualization)/urdf/robotiq_arg2f_85_model_macro.xacro" />
+<!-- arm parameters -->
+<xacro:include filename="$(find ur_description)/urdf/inc/ur5_macro.xacro"/>
+<xacro:ur5_robot prefix="ur5_"
+  transmission_hw_interface="(arg transmission_hw_interface)"
+  kinematics_parameters_file="$(arg kinematics_config_ur5)"
+  joint_limits_parameters_file="$(arg joint_limits_config_ur5)"
+/>
 <joint name="ur5_joint" type="fixed">
   <parent link="shopdesk" />
   <child  link = "ur5_base_link" />
-  <origin xyz="0.7    -0.2   0.0" rpy="0 0 ${0*pi-0.2}" />
+  <origin xyz="0.7    -0.2   0.0" rpy="0 0 0" />
 </joint>
-<xacro:include filename="$(find ur_description)/urdf/inc/ur5_macro.xacro"/>
-<xacro:ur5_robot prefix="ur5_"
-   transmission_hw_interface="$(arg transmission_hw_interface)"
-/>
 <xacro:robotiq_ft300 parent="ur5_tool0" prefix="">
   <origin xyz="0 0 0" rpy="0 0 0"/>
@@ -28,5 +32,5 @@
   <parent link="ur5_tool0" />
   <child  link = "tip" />
-  <origin xyz="0 0 0.2078" rpy="0 0 0" />
+  <origin xyz="0 0 0.14" rpy="0 0 0" />
 </joint>
 <gazebo reference="ur5_tool0">>
@@ -40,4 +44,4 @@
   </plugin>
 </gazebo>
-</xacro:macro>
+<!--/xacro:macro-->
 </robot>
